File: PCBs/Autism Ray/autism_ray_board.sch (EAGLE design)
At the start: 5 parts, among them U1 RFM95W-915S2, U2 RASPBERRY_PICOSMD

Commit message: Update PCB
Parts:
- added X2: (no value), adafruit:SMACONNECTOR_EDGE_UFL
Connections:
- net ANT: now also X2.ANT
- net GND: now also X2.GND1, X2.GND2, X2.GND3, X2.GND4
Other:
- moved on the sheet: CN1, U2
Changed lines of the file:
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@@
 <part name="GND3" library="supply1" library_urn="urn:adsk.eagle:library:371" deviceset="GND" device=""/>
 <part name="FRAME1" library="frames" library_urn="urn:adsk.eagle:library:229" deviceset="A3L-LOC" device=""/>
+<part name="X2" library="adafruit" library_urn="urn:adsk.eagle:library:420" deviceset="SMACONNECTOR" device="_EDGE_UFL" package3d_urn="urn:adsk.eagle:package:6240947/1"/>
 </parts>
 <sheets>
@@
 <attribute name="VALUE" x="-64.135" y="69.85" size="1.778" layer="96"/>
 </instance>
-<instance part="U2" gate="U$1" x="-104.14" y="114.3" smashed="yes">
-<attribute name="NAME" x="-116.8555" y="153.7146" size="2.54388125" layer="95"/>
-<attribute name="VALUE" x="-116.8469" y="72.3686" size="2.54171875" layer="96"/>
+<instance part="U2" gate="U$1" x="-106.68" y="114.3" smashed="yes">
+<attribute name="NAME" x="-119.3955" y="153.7146" size="2.54388125" layer="95"/>
+<attribute name="VALUE" x="-119.3869" y="72.3686" size="2.54171875" layer="96"/>
 </instance>
 <instance part="X1" gate="G$1" x="20.32" y="53.34" smashed="yes" rot="R90">
@@
 <attribute name="VALUE" x="30.48" y="50.8" size="1.27" layer="96" rot="R90"/>
 </instance>
-<instance part="CN1" gate="G$1" x="-167.64" y="182.88" smashed="yes" rot="R90">
-<attribute name="NAME" x="-168.275" y="186.69" size="1.778" layer="95" rot="R180"/>
-<attribute name="VALUE" x="-162.56" y="176.53" size="1.778" layer="96" rot="R90"/>
+<instance part="CN1" gate="G$1" x="-33.02" y="180.34" smashed="yes" rot="R90">
+<attribute name="NAME" x="-33.655" y="184.15" size="1.778" layer="95" rot="R180"/>
+<attribute name="VALUE" x="-27.94" y="173.99" size="1.778" layer="96" rot="R90"/>
 </instance>
-<instance part="SUPPLY1" gate="G$1" x="-142.24" y="182.88" smashed="yes">
-<attribute name="VALUE" x="-142.24" y="185.674" size="1.778" layer="96" align="bottom-center"/>
+<instance part="SUPPLY1" gate="G$1" x="-7.62" y="180.34" smashed="yes">
+<attribute name="VALUE" x="-7.62" y="183.134" size="1.778" layer="96" align="bottom-center"/>
 </instance>
 <instance part="GND1" gate="1" x="71.12" y="50.8" smashed="yes" rot="R90">
@@
 <attribute name="VALUE" x="-73.406" y="149.86" size="1.778" layer="96" rot="R180" align="bottom-center"/>
 </instance>
-<instance part="GND2" gate="1" x="-190.5" y="182.88" smashed="yes" rot="R180">
-<attribute name="VALUE" x="-187.96" y="185.42" size="1.778" layer="96" rot="R180"/>
+<instance part="GND2" gate="1" x="-55.88" y="180.34" smashed="yes" rot="R180">
+<attribute name="VALUE" x="-53.34" y="182.88" size="1.778" layer="96" rot="R180"/>
 </instance>
 <instance part="GND3" gate="1" x="-73.66" y="60.96" smashed="yes">
@@
 <attribute name="LAST_DATE_TIME" x="92.71" y="-7.62" size="2.286" layer="94"/>
 <attribute name="SHEET" x="106.045" y="-12.7" size="2.54" layer="94"/>
+</instance>
+<instance part="X2" gate="G$1" x="27.94" y="40.64" smashed="yes" rot="R270">
+<attribute name="NAME" x="30.48" y="33.02" size="1.27" layer="95" rot="R270"/>
+<attribute name="VALUE" x="27.94" y="33.02" size="1.27" layer="95" rot="R270"/>
 </instance>
 </instances>
@@
 <wire x1="20.32" y1="83.82" x2="22.86" y2="83.82" width="0.1524" layer="91"/>
 <label x="15.24" y="63.5" size="1.778" layer="95"/>
+<pinref part="X2" gate="G$1" pin="ANT"/>
+<wire x1="27.94" y1="48.26" x2="20.32" y2="48.26" width="0.1524" layer="91"/>
+<wire x1="20.32" y1="48.26" x2="20.32" y2="58.42" width="0.1524" layer="91"/>
+<junction x="20.32" y="58.42"/>
 </segment>
 </net>
@@
 <pinref part="GND2" gate="1" pin="GND"/>
 <pinref part="CN1" gate="G$1" pin="1"/>
-<wire x1="-190.5" y1="180.34" x2="-170.18" y2="180.34" width="0.1524" layer="91"/>
-<label x="-185.42" y="180.34" size="1.778" layer="95"/>
+<wire x1="-55.88" y1="177.8" x2="-35.56" y2="177.8" width="0.1524" layer="91"/>
+<label x="-50.8" y="177.8" size="1.778" layer="95"/>
 </segment>
 <segment>
 <pinref part="U2" gate="U$1" pin="GND"/>
 <pinref part="LS1" gate="G$1" pin="-"/>
-<wire x1="-86.36" y1="78.74" x2="-73.66" y2="78.74" width="0.1524" layer="91"/>
+<wire x1="-88.9" y1="78.74" x2="-73.66" y2="78.74" width="0.1524" layer="91"/>
 <pinref part="GND3" gate="1" pin="GND"/>
 <wire x1="-73.66" y1="78.74" x2="-58.42" y2="78.74" width="0.1524" layer="91"/>
@@
 <wire x1="68.58" y1="63.5" x2="68.58" y2="50.8" width="0.1524" layer="91"/>
 <pinref part="X1" gate="G$1" pin="GND@1"/>
-<wire x1="27.94" y1="50.8" x2="68.58" y2="50.8" width="0.1524" layer="91"/>
+<wire x1="27.94" y1="50.8" x2="35.56" y2="50.8" width="0.1524" layer="91"/>
 <junction x="68.58" y="50.8"/>
+<pinref part="X2" gate="G$1" pin="GND2"/>
+<pinref part="X2" gate="G$1" pin="GND1"/>
+<wire x1="35.56" y1="50.8" x2="68.58" y2="50.8" width="0.1524" layer="91"/>
+<wire x1="35.56" y1="38.1" x2="35.56" y2="43.18" width="0.1524" layer="91"/>
+<wire x1="35.56" y1="43.18" x2="35.56" y2="50.8" width="0.1524" layer="91"/>
+<junction x="35.56" y="43.18"/>
+<junction x="35.56" y="50.8"/>
+<pinref part="X2" gate="G$1" pin="GND4"/>
+<pinref part="X2" gate="G$1" pin="GND3"/>
+<wire x1="20.32" y1="38.1" x2="20.32" y2="43.18" width="0.1524" layer="91"/>
+<wire x1="20.32" y1="38.1" x2="35.56" y2="38.1" width="0.1524" layer="91"/>
+<junction x="20.32" y="38.1"/>
+<junction x="35.56" y="38.1"/>
 </segment>
 </net>
@@
 <segment>
 <pinref part="U2" gate="U$1" pin="GP16"/>
-<wire x1="-86.36" y1="91.44" x2="-15.24" y2="91.44" width="0.1524" layer="91"/>
+<wire x1="-88.9" y1="91.44" x2="-15.24" y2="91.44" width="0.1524" layer="91"/>
 <wire x1="-15.24" y1="91.44" x2="-15.24" y2="96.52" width="0.1524" layer="91"/>
 <pinref part="U1" gate="G$1" pin="MISO"/>
@@
 <segment>
 <pinref part="U2" gate="U$1" pin="GP18"/>
-<wire x1="-86.36" y1="99.06" x2="-17.78" y2="99.06" width="0.1524" layer="91"/>
+<wire x1="-88.9" y1="99.06" x2="-17.78" y2="99.06" width="0.1524" layer="91"/>
 <wire x1="-17.78" y1="99.06" x2="-17.78" y2="93.98" width="0.1524" layer="91"/>
 <pinref part="U1" gate="G$1" pin="SCK"/>
@@
 <segment>
 <pinref part="U2" gate="U$1" pin="GP19"/>
-<wire x1="-86.36" y1="101.6" x2="43.18" y2="101.6" width="0.1524" layer="91"/>
+<wire x1="-88.9" y1="101.6" x2="43.18" y2="101.6" width="0.1524" layer="91"/>
 <wire x1="43.18" y1="101.6" x2="43.18" y2="96.52" width="0.1524" layer="91"/>
 <pinref part="U1" gate="G$1" pin="MOSI"/>
@@
 <pinref part="U2" gate="U$1" pin="GP22"/>
 <wire x1="-48.26" y1="78.74" x2="-48.26" y2="111.76" width="0.1524" layer="91"/>
-<wire x1="-48.26" y1="111.76" x2="-86.36" y2="111.76" width="0.1524" layer="91"/>
+<wire x1="-48.26" y1="111.76" x2="-88.9" y2="111.76" width="0.1524" layer="91"/>
 <label x="-60.96" y="111.76" size="1.778" layer="95"/>
 </segment>
@@
 <wire x1="-81.28" y1="83.82" x2="-81.28" y2="93.98" width="0.1524" layer="91"/>
 <pinref part="U2" gate="U$1" pin="GP17"/>
-<wire x1="-81.28" y1="93.98" x2="-86.36" y2="93.98" width="0.1524" layer="91"/>
+<wire x1="-81.28" y1="93.98" x2="-88.9" y2="93.98" width="0.1524" layer="91"/>
 <label x="-25.4" y="83.82" size="1.778" layer="95"/>
 </segment>
@@
 <segment>
 <pinref part="U2" gate="U$1" pin="GP28"/>
-<wire x1="-86.36" y1="124.46" x2="2.54" y2="124.46" width="0.1524" layer="91"/>
+<wire x1="-88.9" y1="124.46" x2="2.54" y2="124.46" width="0.1524" layer="91"/>
 <wire x1="2.54" y1="124.46" x2="2.54" y2="86.36" width="0.1524" layer="91"/>
 <pinref part="U1" gate="G$1" pin="RESET"/>
@@
 <segment>
 <pinref part="U2" gate="U$1" pin="3V3(OUT)"/>
-<wire x1="-86.36" y1="144.78" x2="-83.82" y2="144.78" width="0.1524" layer="91"/>
+<wire x1="-88.9" y1="144.78" x2="-83.82" y2="144.78" width="0.1524" layer="91"/>
 <wire x1="-83.82" y1="144.78" x2="-83.82" y2="129.54" width="0.1524" layer="91"/>
 <wire x1="-83.82" y1="129.54" x2="58.42" y2="129.54" width="0.1524" layer="91"/>
@@
 <pinref part="CN1" gate="G$1" pin="2"/>
 <pinref part="SUPPLY1" gate="G$1" pin="VCC"/>
-<wire x1="-167.64" y1="180.34" x2="-142.24" y2="180.34" width="0.1524" layer="91"/>
-<wire x1="-142.24" y1="180.34" x2="-142.24" y2="182.88" width="0.1524" layer="91"/>
-<label x="-157.48" y="180.34" size="1.778" layer="95"/>
+<wire x1="-33.02" y1="177.8" x2="-7.62" y2="177.8" width="0.1524" layer="91"/>
+<wire x1="-7.62" y1="177.8" x2="-7.62" y2="180.34" width="0.1524" layer="91"/>
+<label x="-22.86" y="177.8" size="1.778" layer="95"/>
 </segment>
 <segment>
 <pinref part="U2" gate="U$1" pin="VSYS"/>
 <pinref part="SUPPLY2" gate="G$1" pin="VCC"/>
-<wire x1="-86.36" y1="147.32" x2="-73.66" y2="147.32" width="0.1524" layer="91"/>
+<wire x1="-88.9" y1="147.32" x2="-73.66" y2="147.32" width="0.1524" layer="91"/>
 </segment>
 </net>
