File: PCBs/Tax Fraud 2/tax fraud 2.sch (EAGLE design)
At the start: 8 parts, among them J1 USB4105-GF-A, U1 RFM95W-915S2

Commit message: TF2 autosave
Parts:
- removed CN1: (no value), adafruit:JST_2PIN-SMT-RA
- removed J1: USB4105-GF-A, USB-C Adafruit USB4105-GF-A:USB4105-GF-A
- removed J2: (no value), SparkFun-Connectors:QWIIC_CONNECTORJS-1MM
- removed LS1: AI-1223-TWT-12V-R, buzzer:AI-1223-TWT-12V-R
- added BEEPER: AI-1223-TWT-12V-R, buzzer:AI-1223-TWT-12V-R
- added BMP3XX: ADAFRUIT_INDUSTRIES_3966ADAFRUIT_INDUSTRIES_3966_0_0, BMP388 Breakout:ADAFRUIT_INDUSTRIES_3966ADAFRUIT_INDUSTRIES_3966_0_0
- added JST-PH: (no value), adafruit:JST_2PIN-SMT-RA
- added QWIIC: (no value), SparkFun-Connectors:QWIIC_CONNECTORJS-1MM
- added UFL: (no value), adafruit:ANTENNA_U.FL
- added USB-C: USB4105-GF-A, USB-C Adafruit USB4105-GF-A:USB4105-GF-A
Connections:
- new net ANT: U1.ANT, UFL.SIGNAL
- new net CS: U$1.IO5, U1.NSS
- new net DN: U$1.D-, USB-C.DN1, USB-C.DN2
- new net DP: U$1.D+, USB-C.DP1, USB-C.DP2
- new net GND: BEEPER.-, BMP3XX.GND, JST-PH.1, QWIIC.GND, R1.2, R2.1, U$1.GND, U1.GND, UFL.GND@0, UFL.GND@1, USB-C.GND
- new net GPIO9: BEEPER.+, U$1.GPIO9
- new net MISO: U$1.IO19, U1.MISO
- new net MOSI: U$1.IO23, U1.MOSI
- new net N$4: U$1.GPIO36
- new net RST: U$1.IO0, U1.RESET
- new net SCK: U$1.IO18, U1.SCK
- new net SCL: BMP3XX.SCK/SCL, QWIIC.SCL, U$1.IO22
- new net SDA: BMP3XX.SDI/SDA, QWIIC.SDA, U$1.IO21
- new net VBAT: JST-PH.2, U$1.VBAT
- new net VCC: BMP3XX.VIN, QWIIC.VCC, U$1.3V3, U1.3.3V
- new net VIN: U$1.5V, USB-C.VBUS
- net N$1: now also R1.1, USB-C.CC2; no longer J1.CC1, R1.2
- net N$2: now also USB-C.CC1; no longer J1.CC2
Other:
- moved on the sheet: R1, R2, U1
