File: PCBs/Tax Fraud 2/Eagle Draft/tax fraud 2.sch (EAGLE design)
At the start: 10 parts, among them U1 RFM95W-915S2

Commit message: Tax Fraud v2 PCB
Parts:
- removed QWIIC: (no value), SparkFun-Connectors:QWIIC_CONNECTORJS-1MM
- removed R1, R2: CR1206-JW-512ELF, resis CR1206-JW-512ELF:CR1206-JW-512ELF
- added D1: 1655, 5050 NeoPixel:1655
- added J1: (no value), SparkFun-Connectors:QWIIC_CONNECTORJS-1MM
- added U2: (no value), adafruit:GPS_FGPMMOPA6H
Connections:
- removed net GPIO9: BEEPER.+, U$1.GPIO9
- removed net N$1: R1.1, USB-C.CC2
- removed net N$2: R2.2, USB-C.CC1
- removed net N$4: U$1.GPIO36
- new net BEEP: BEEPER.+, U$1.IO35
- new net FIX: U$1.GPIO39, U2.3D-FIX
- new net NEO: D1.DIN, U$1.GPIO38
- new net RX: U$1.TX, U2.RX
- new net TX: U$1.RX, U2.TX
- new net VBACK: U2.VBACKUP
- net GND: now also D1.VSS, J1.GND, U2.GND@1, U2.GND@2, U2.GND@3, U2.GND@4; no longer QWIIC.GND, R1.2, R2.1
- net SCL: now also J1.SCL; no longer QWIIC.SCL
- net SDA: now also J1.SDA; no longer QWIIC.SDA
- net VCC: now also J1.VCC, U2.VCC; no longer QWIIC.VCC
- net VIN: now also D1.VDD
Other:
- moved on the sheet: BMP3XX
