File: PCBs/ChungRF/ChungRF.kicad_pcb (KiCad board)
At the start: 4 copper layers, 28.4 x 53.3 mm, 15 parts, among them J1 Conn_Coaxial, J2 Conn_01x09_Socket, U1 E22-900M30S

Commit message: Update ChungRF
Parts:
- moved R1 27.5 mm to (161.5, 91.3)
- moved R2 27.5 mm to (161.5, 93.8)
- moved C1 27.5 mm to (156.6, 102.2)
- moved C2 27.5 mm to (158.1, 102.2)
- moved H3 27.5 mm to (165.5, 64.4)
- moved J1 27.5 mm to (172.5, 65.1)
- moved J2 27.5 mm to (165.5, 110.9)
- moved TP2 27.5 mm to (164.6, 98.4)
- moved TP3 27.5 mm to (157.9, 91.3)
- moved TP4 27.5 mm to (157.9, 93.8)
- moved TP5 27.5 mm to (157.9, 96.4)
- moved TP1 27.5 mm to (160.4, 101.5)
- moved U1 27.5 mm to (165.5, 87.4)
- moved H1 27.3 mm to (154.5, 111.4)
- moved H2 27.3 mm to (176.5, 111.4)
Routing:
- net /TXEN: track 6.62 -> 7.18 mm
- net /RXEN: track 6.62 -> 7.18 mm
- net GND: track 31.8 -> 31.7 mm, vias 44 -> 96
Other:
- board size 28.4 x 53.3 mm -> 28.4 x 53.4 mm
- board text added: "R1 5-24"
- board text added: "{ "ViaStitching": "0.2", "stitch_zone_0": { "HSpacing": "1", "VSpacing": "1", "Clearance": "0", "Randomize": false } }"
- board text added: "{ "ViaStitching": "0.2", "stitch_zone_0": { "HSpacing": "1", "VSpacing": "1", "Clearance": "0", "Randomize": true } }"
- board text added: "{ "ViaStitching": "0.2", "stitch_zone_0": { "HSpacing": "1", "VSpacing": "4", "Clearance": "0", "Randomize": false } }"
- board text removed: "Modify footprint to have less pad sticking out? Rename to ChungRF add chungus or other image Use 0402 caps, or remove them"

Commit message: Fix impedance
Other:
- board text added: "Switch to 10 pin con for extra ground pin"

Commit message: Finalize design, add gerbers
Routing:
- net GND: track 31.7 -> 34.6 mm, vias 96 -> 99
Other:
- board text added: "Chungus Aerospace"
- board text added: "DIO2"
- board text added: "GND"
- board text added: "R1 5-2024"
- board text added: "RXEN"
- board text added: "TXEN"
- board text added: "VCC"
- board text removed: "R1 5-24"
- board text removed: "Switch to 10 pin con for extra ground pin"

Commit message: Update ChungRF, add software tests
Other:
- board text added: "R2 5-2024"
- board text removed: "R1 5-2024"
Changed lines of the file:
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@@
 	(title_block
 		(title "ChungRF")
-		(date "2024-05-14")
-		(rev "R1")
+		(date "2024-05-23")
+		(rev "R2")
 		(company "Chungus Aerospace")
 	)
@@
 		(layer "Edge.Cuts")
 	)
-	(gr_text "R1\n5-2024"
+	(gr_text "R2\n5-2024"
 		(at 155.2 66.9 0)
 		(layer "B.SilkS")
@@
 			(justify bottom mirror)
 		)
-		(render_cache "R1\n5-2024" 0
+		(render_cache "R2\n5-2024" 0
 			(polygon
 				(pts
@@
 			(polygon
 				(pts
-					(xy 154.999231 63.760865) (xy 154.942869 63.736259) (xy 154.897236 63.714556) (xy 154.844626 63.686933)
-					(xy 154.793481 63.656817) (xy 154.743876 63.624651) (xy 154.696468 63.590872) (xy 154.649601 63.552656)
-					(xy 154.612644 63.517013) (xy 154.437082 63.517013) (xy 154.437082 64.68) (xy 154.688555 64.68)
-					(xy 154.688555 63.835896) (xy 154.738666 63.867031) (xy 154.79393 63.895591) (xy 154.801688 63.899204)
-					(xy 154.855696 63.922622) (xy 154.912192 63.944475) (xy 154.923321 63.948443)
+					(xy 154.279985 63.828862) (xy 154.285588 63.887393) (xy 154.302396 63.943734) (xy 154.305484 63.951081)
+					(xy 154.332463 64.004859) (xy 154.36614 64.056834) (xy 154.371137 64.063628) (xy 154.408491 64.110287)
+					(xy 154.449772 64.155375) (xy 154.462288 64.167969) (xy 154.506318 64.210869) (xy 154.549675 64.251862)
+					(xy 154.561939 64.263224) (xy 154.606084 64.305195) (xy 154.61704 64.31598) (xy 154.658112 64.358296)
+					(xy 154.673607 64.375184) (xy 154.712161 64.41957) (xy 154.721674 64.431165) (xy 154.747759 64.473663)
+					(xy 154.244521 64.473663) (xy 154.244521 64.68) (xy 155.024437 64.68) (xy 155.027954 64.633105)
+					(xy 155.027954 64.592658) (xy 155.024286 64.534104) (xy 155.012033 64.474949) (xy 155.001869 64.44494)
+					(xy 154.975759 64.388007) (xy 154.94359 64.334665) (xy 154.933286 64.320083) (xy 154.894281 64.270764)
+					(xy 154.854344 64.227579) (xy 154.838031 64.211639) (xy 154.794884 64.17068) (xy 154.752123 64.12972)
+					(xy 154.732518 64.110816) (xy 154.688592 64.068683) (xy 154.656608 64.037836) (xy 154.615598 63.995544)
+					(xy 154.594179 63.970718) (xy 154.560327 63.921644) (xy 154.551974 63.905359) (xy 154.536971 63.84724)
+					(xy 154.536733 63.838827) (xy 154.546007 63.77918) (xy 154.578938 63.73478) (xy 154.632818 63.71037)
+					(xy 154.683572 63.704591) (xy 154.743405 63.711379) (xy 154.768862 63.718953) (xy 154.824421 63.743463)
+					(xy 154.841255 63.752951) (xy 154.890181 63.785803) (xy 154.897822 63.791933) (xy 154.933286 63.823)
+					(xy 155.058143 63.65711) (xy 155.009393 63.616255) (xy 154.955836 63.580151) (xy 154.903522 63.55172)
+					(xy 154.885219 63.543098) (xy 154.828524 63.521421) (xy 154.769557 63.506838) (xy 154.708317 63.49935)
+					(xy 154.673314 63.498255) (xy 154.611822 63.500545) (xy 154.55066 63.508353) (xy 154.496287 63.521702)
+					(xy 154.440153 63.543897) (xy 154.389439 63.574832) (xy 154.373774 63.587648) (xy 154.33425 63.631547)
+					(xy 154.305802 63.683561) (xy 154.302846 63.691109) (xy 154.286437 63.751739) (xy 154.280186 63.814603)
 				)
 			)

Commit message: ChungRF R2
Parts:
- removed H3: MountingHole, MountingHole:MountingHole_2.7mm_M2.5_Pad_Via
- removed TP1: VCC, TestPoint:TestPoint_Pad_D1.5mm
- removed TP2: GND, TestPoint:TestPoint_Pad_D1.5mm
- removed TP3: RXEN, TestPoint:TestPoint_Pad_D1.5mm
- removed TP4: TXEN, TestPoint:TestPoint_Pad_D1.5mm
- removed TP5: DIO2, TestPoint:TestPoint_Pad_D1.5mm
- added C3: 10uF, Capacitor_SMD:C_0603_1608Metric, B.Cu at (154.9, 98.7)
- added U1: KB2040, besser_footprints:Adafuit-KB2040-SMD, B.Cu at (168.1, 96.7)
- H1, H2: value MountingHole -> 2.7mm_M2.5_Pad_Via
- J1: value Conn_Coaxial -> JST-SM04B-SRSS; footprint besser_footprints:CON-SMA-EDGE-S -> besser_footprints:JST_SH_SM04B-SRSS-TB_1x04-1MP_P1.00mm_Horizontal
- J2: value Conn_01x09_Socket -> Conn_Coaxial; footprint Connector_JST:JST_SH_SM09B-SRSS-TB_1x09-1MP_P1.00mm_Horizontal -> besser_footprints:CONSMA003.062
- R1, R2: value 100k -> 10k
- moved H1 48.0 mm to (165.5, 64.7), turned to 0 degrees
- moved J2 46.2 mm to (172.6, 65.2)
- moved J1 45.9 mm to (165.5, 110.5)
- moved H2 22.0 mm to (154.5, 110.6), turned to 0 degrees
- moved R2 6.55 mm to (154.9, 93.8)
- moved R1 6.55 mm to (154.9, 91.3)
- moved C2 3.80 mm to (154.9, 100.2), turned to 0 degrees
- moved C1 1.78 mm to (154.9, 101.7), turned to 0 degrees
- renumbered U1 to U2
Connections:
- C1 pad 1: VCC -> VBUS
- C2 pad 1: VCC -> VBUS
- J1 pad 1: /RF_ANT -> GND
- J1 pad 2: GND -> VBUS
- J2 pad 1: VCC -> /RF_ANT
- U2 pad 10: VCC -> VBUS
- U2 pad 9: VCC -> VBUS
Routing:
- net VBUS: track 0.00 -> 31.3 mm, vias 0 -> 3
- net /NSS: track 29.9 -> 11.9 mm, vias 0 -> 1
- net VCC: track 17.2 -> 0.00 mm, vias 2 -> 0
- net /SCK: track 27.0 -> 11.8 mm, vias 0 -> 1
- net /MOSI: track 24.0 -> 11.4 mm, vias 0 -> 1
- net /MISO: track 21.1 -> 11.4 mm, vias 0 -> 1
- net /CARFIO_MOSI: track 0.00 -> 9.41 mm, vias 0 -> 1
- net /CARFIO_MISO: track 0.00 -> 8.08 mm, vias 0 -> 1
- net /NRST: track 17.7 -> 11.5 mm, vias 0 -> 1
- net GND: track 34.6 -> 39.3 mm, vias 99 -> 79
- net /RXEN: track 7.18 -> 3.52 mm
- net /BUSY: track 14.8 -> 11.4 mm, vias 0 -> 1
- net /TXEN: track 7.18 -> 4.88 mm
- net /DIO2: track 4.40 -> 5.91 mm
- net /DIO1: track 11.8 -> 11.4 mm, vias 0 -> 1
- added copper zone on B.Cu, net VBUS
Other:
- board size 28.4 x 53.4 mm -> 28.4 x 52.3 mm
- board text added: "ANT"
- board text added: "CARFIO"
- board text added: "R2 6-2024"
- board text removed: "Chungus Aerospace"
- board text removed: "DIO2"
- board text removed: "EBYTE E22-900M30S"
- board text removed: "GND"
- board text removed: "R2 5-2024"
- board text removed: "RXEN"
- board text removed: "TXEN"
- board text removed: "VCC"

Commit message: ChungRF R3
Connections:
- net /CARFIO_MISO renamed /CARFIO_SDA
- net /CARFIO_MOSI renamed /CARFIO_SCL
- U1 pad 14: /NSS -> unconnected-(U1-D10-Pad14)
- U1 pad 15: /SCK -> /MOSI
- U1 pad 16: /MOSI -> /MISO
- U1 pad 17: /MISO -> /SCK
- U1 pad 18: /NRST -> unconnected-(U1-A0-Pad18)
- U1 pad 19: /BUSY -> unconnected-(U1-A1-Pad19)
- U1 pad 20: /DIO1 -> unconnected-(U1-A2-Pad20)
- U1 pad 6: unconnected-(U1-D2-Pad6) -> /DIO1
- U1 pad 7: /DIO2 -> /NSS
- U1 pad 8: unconnected-(U1-D4-Pad8) -> /NRST
- U1 pad 9: unconnected-(U1-D5-Pad9) -> /BUSY
- U2 pad 8: /DIO2 -> unconnected-(U2-DIO2-Pad8)
Routing:
- net /NSS: track 11.9 -> 25.6 mm
- net /BUSY: track 11.4 -> 21.2 mm
- net /DIO1: track 11.4 -> 19.1 mm
- net /NRST: track 11.5 -> 19.1 mm
- net /SCK: track 11.8 -> 5.75 mm
- net /DIO2: track 5.91 -> 0.00 mm, vias 1 -> 0
- net /MOSI: track 11.4 -> 15.1 mm
- net /MISO: track 11.4 -> 13.3 mm
- net GND: vias 79 -> 84
Other:
- board text added: "R3 10-2024"
- board text removed: "R2 6-2024"

Commit message: Clean Tracks, add Gerber files
Parts:
- removed R1, R2: 10k, Capacitor_SMD:C_0603_1608Metric
Connections:
- U1 pad 11: unconnected-(U1-D7-Pad11) -> /NSS
- U1 pad 12: unconnected-(U1-D8-Pad12) -> /TXEN
- U1 pad 13: unconnected-(U1-D9-Pad13) -> /RXEN
- U1 pad 7: /NSS -> unconnected-(U1-D3-Pad7)
Routing:
- net /RXEN: track 3.32 -> 17.4 mm
- net /TXEN: track 4.68 -> 16.6 mm
- net /NSS: track 25.6 -> 18.8 mm
- net GND: track 39.3 -> 37.4 mm, vias 84 -> 85
- net /MOSI: track 15.1 -> 16.2 mm
- net /BUSY: track 21.2 -> 22.3 mm

Commit message: ChungRF R3
Parts:
- added J3: uFL, Connector_Coaxial:U.FL_Hirose_U.FL-R-SMT-1_Vertical, B.Cu at (160.4, 65.3)
- added R1: 5.1k, Capacitor_SMD:C_0603_1608Metric, B.Cu at (165.5, 77.5)
- added R2: 5.1k, Capacitor_SMD:C_0603_1608Metric, B.Cu at (168.6, 77.5)
- added U3: ZOE-M8Q, RF_GPS:ublox_ZOE_M8, B.Cu at (159.9, 69.8)
- H1, H2: value 2.7mm_M2.5_Pad_Via -> 2.7mm_M2.5_Pad; footprint MountingHole:MountingHole_2.7mm_M2.5_Pad_Via -> besser_footprints:M2.5_2.7mm_hole
- moved H1 0.35 mm to (165.9, 64.6)
- moved H2 0.16 mm to (154.5, 110.8)
Connections:
- U1 pad 10: unconnected-(U1-D6-Pad10) -> /GNSS_SCL
- U1 pad 14: unconnected-(U1-D10-Pad14) -> /GNSS_SDA
- U1 pad 22: unconnected-(U1-3v3-Pad22) -> +3V3
Routing:
- net +3V3: track 0.00 -> 51.3 mm, vias 0 -> 3
- net /GNSS_SCL: track 0.00 -> 26.8 mm, vias 0 -> 2
- net /GNSS_SDA: track 0.00 -> 26.1 mm
- net GND: track 37.4 -> 53.2 mm, vias 85 -> 100
- net /RXEN: track 17.4 -> 13.8 mm
- net /TXEN: track 16.6 -> 13.7 mm
- net /RF_GNSS: track 0.00 -> 1.48 mm
Other:
- board size 28.4 x 52.3 mm -> 28.3 x 52.3 mm
- board text added: "GNSS"
- board text added: "R3 11-2024"
- board text added: "RDIO"
- board text removed: "ANT"
- board text removed: "JLCJLCJLCJLC"
- board text removed: "R3 10-2024"
