File: PCBs/ChungRF/ChungRF.kicad_pcb (KiCad board)
At the start: 4 copper layers, 28.3 x 52.3 mm, 13 parts, among them J1 JST-SM04B-SRSS, J2 Conn_Coaxial, J3 uFL, U1 KB2040, U2 E22-900M30S, U3 ZOE-M8Q

Commit message: ChungRF R4 - Fix GNSS I2C bus
Connections:
- U1 pad 10: /GNSS_SCL -> unconnected-(U1-D6-Pad10)
- U1 pad 7: unconnected-(U1-D3-Pad7) -> /GNSS_SCL
Routing:
- net /GNSS_SCL: track 26.8 -> 34.5 mm
Changed lines of the file:
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@@
 	(title_block
 		(title "ChungRF")
-		(date "2024-11-06")
-		(rev "R3")
+		(date "2024-11-13")
+		(rev "R4")
 		(company "Chungus Aerospace")
 	)
@@
 	(net 22 "/CARFIO_SCL")
 	(net 23 "/CARFIO_SDA")
-	(net 24 "unconnected-(U1-D3-Pad7)")
+	(net 24 "unconnected-(U1-D6-Pad10)")
 	(net 25 "+3V3")
 	(net 26 "unconnected-(U3-TIMEPULSE-PadC3)")
@@
 			(layers "B.Cu" "B.Paste" "B.Mask")
 			(roundrect_rratio 0.125)
-			(net 24 "unconnected-(U1-D3-Pad7)")
+			(net 52 "/GNSS_SCL")
 			(pinfunction "D3")
-			(pintype "bidirectional+no_connect")
+			(pintype "bidirectional")
 		)
 		(pad "8" smd roundrect
@@
 			(layers "B.Cu" "B.Paste" "B.Mask")
 			(roundrect_rratio 0.125)
-			(net 52 "/GNSS_SCL")
+			(net 24 "unconnected-(U1-D6-Pad10)")
 			(pinfunction "D6")
-			(pintype "bidirectional")
+			(pintype "bidirectional+no_connect")
 		)
 		(pad "11" smd roundrect
@@
 	)
 	(segment
-		(start 166.3 79)
-		(end 166.3 84.3)
+		(start 166.275 83.975)
+		(end 166.275 79.025)
+		(width 0.2)
+		(layer "F.Cu")
+		(net 52)
+	)
+	(segment
+		(start 166.2 79)
+		(end 166.3 79.1)
 		(width 0.2)
 		(layer "F.Cu")
@@
 	)
 	(segment
-		(start 166.3 84.3)
-		(end 162.45 88.15)
+		(start 162.2 88.05)
+		(end 166.275 83.975)
 		(width 0.2)
 		(layer "F.Cu")
@@
 	)
 	(segment
-		(start 162.45 88.15)
-		(end 162.25 88.35)
+		(start 162.2 95.95)
+		(end 162.2 88.05)
+		(width 0.2)
+		(layer "F.Cu")
+		(net 52)
+	)
+	(segment
+		(start 166.275 79)
+		(end 166.25 79.025)
 		(width 0.2)
 		(layer "F.Cu")
@@
 	)
 	(via
-		(at 162.25 88.35)
+		(at 166.275 79)
 		(size 0.6)
 		(drill 0.3)
@@
 	)
 	(via
-		(at 166.3 79)
+		(at 162.2 95.95)
 		(size 0.6)
 		(drill 0.3)
@@
 	)
 	(segment
-		(start 166.3 79)
-		(end 166.3 77.575)
-		(width 0.2)
-		(layer "B.Cu")
-		(net 52)
-	)
-	(segment
-		(start 159.35 89.03)
-		(end 161.57 89.03)
+		(start 162.140918 68.33)
+		(end 166.3 72.489082)
 		(width 0.2)
 		(layer "B.Cu")
@@
 	)
 	(segment
-		(start 162.140918 68.33)
-		(end 166.3 72.489082)
+		(start 162.2 95.95)
+		(end 161.5 96.65)
 		(width 0.2)
 		(layer "B.Cu")
@@
 	)
 	(segment
-		(start 161.57 89.03)
-		(end 162.25 88.35)
+		(start 166.275 79)
+		(end 166.275 77.55)
 		(width 0.2)
 		(layer "B.Cu")
@@
 	)
 	(segment
-		(start 166.3 77.575)
-		(end 166.275 77.55)
+		(start 161.5 96.65)
+		(end 159.35 96.65)
 		(width 0.2)
 		(layer "B.Cu")
